File: hardware/rfid-emulator.sch (KiCad schematic (older format))
At the start: 102 parts, among them J1 AVR-JTAG-10, J2 Micro_USB, J3 OSTTC020162, Q1 2N3904, Q2 2N3906, Q3 2N3906, Q4 IRLML6344TRPBF, Q5 IRLML6344TRPBF, SW1 EN11-HSM1BF20, U1 NHD-C0216CiZ-FSW-FBW-3V3, U2 LT8613, U3 ATmega64A-AU, U4 MCP73832-2-OT, U5 LF33_TO252, U6 FT230XS, U7 LM324DT, Y1 ECS-160-20-5PX-TR

Commit message: Remove unnecessary components and apply fixes from V0.1
Parts:
- removed C10: 0.1u, Capacitors_SMD:C_0805_HandSoldering, symbol Device:C_Small
- removed C11: 10p, Capacitors_SMD:C_0805_HandSoldering, symbol Device:C_Small
- removed C2, C7: 1n, Capacitors_SMD:C_0805_HandSoldering, symbol Device:C
- removed C23: 2.2u, rfid-footprints:EEE-1VA2R2NR, symbol Device:CP1
- removed C33: 0.0n, Socket_Strips:Socket_Strip_Straight_1x02_Pitch2.54mm, symbol Device:C
- removed C6: 1u, Capacitors_SMD:C_0805_HandSoldering, symbol Device:C
- removed C9: 0.1u, Capacitors_SMD:C_0805_HandSoldering, symbol Device:C
- removed D1: 1N5817, Diodes_THT:D_DO-41_SOD81_P10.16mm_Horizontal, symbol Diode:1N5817
- removed D3: 1N4148W, Diodes_SMD:D_SOD-123, symbol Diode:1N4148W
- removed D9: D_TVS, rfid-footprints:DO-219AD, symbol Device:D_TVS
- removed FB1: BLM21PG331SN1D, digikey-footprints:0805, symbol dk_Ferrite-Beads-and-Chips:BLM21PG331SN1D
- removed J3: OSTTC020162, digikey-footprints:Term_Block_1x2_P5mm, symbol dk_Terminal-Blocks-Wire-to-Board:OSTTC020162
- removed JP1: CHARGE_SELECT, Jumper:SolderJumper-3_P1.3mm_Open_RoundedPad1.0x1.5mm, symbol Jumper:SolderJumper_3_Bridged12
- removed JP2: ANT_SELECT, Jumper:SolderJumper-3_P1.3mm_Open_RoundedPad1.0x1.5mm, symbol Jumper:SolderJumper_3_Bridged12
- removed L1: 3.9u, rfid-footprints:CDRH6D28, symbol Device:L
- removed Q1: 2N3904, digikey-footprints:TO-92-3, symbol Transistor_BJT:2N3904
- removed Q2, Q3: 2N3906, digikey-footprints:TO-92-3, symbol Transistor_BJT:2N3906
- removed Q4, Q5: IRLML6344TRPBF, digikey-footprints:SOT-23-3, symbol dk_Transistors-FETs-MOSFETs-Single:IRLML6344TRPBF
- removed R1, R2: 10k, Resistors_SMD:R_0805_HandSoldering, symbol Device:R
- removed R4: 60.4k, Resistors_SMD:R_0805_HandSoldering, symbol Device:R
- removed R5: 1M, Resistors_SMD:R_0805_HandSoldering, symbol Device:R
- removed R6: 243k, Resistors_SMD:R_0805_HandSoldering, symbol Device:R
- removed R8: 8m, Resistors_SMD:R_0805_HandSoldering, symbol Device:R
- removed TP1: 5001, digikey-footprints:Test_Point_D1.02mm, symbol dk_Test-Points:5001
- removed TP2, TP3: 5000, digikey-footprints:Test_Point_D1.02mm, symbol dk_Test-Points:5000
- removed TP4, TP5, TP6: 5002, digikey-footprints:Test_Point_D1.02mm, symbol dk_Test-Points:5002
- removed U2: LT8613, Housings_DFN_QFN:QFN-28-1EP_3x6mm_Pitch0.5mm, symbol rfid-emulator:LT8613
- removed U5: LF33_TO252, TO_SOT_Packages_THT:TO-220-3_Horizontal, symbol Regulator_Linear:LF33_TO252
- removed VR1: TL431AIDBZR, digikey-footprints:SOT-23-3, symbol dk_PMIC-Voltage-Reference:TL431AIDBZR
- added C18: 1u, Capacitors_SMD:C_0805_HandSoldering, symbol Device:C
- added Q1: BC847, TO_SOT_Packages_SMD:SOT-23, symbol Transistor_BJT:BC847
- added Q2, Q3: BC857, TO_SOT_Packages_SMD:SOT-23, symbol Transistor_BJT:BC857
- added R7, R8: 4.7k, Resistors_SMD:R_0805_HandSoldering, symbol Device:R_Small
- added U4: MCP1700T-3302E_TT, digikey-footprints:SOT-23-3, symbol dk_PMIC-Voltage-Regulators-Linear:MCP1700T-3302E_TT
- C19: renamed from C24; value 1.8n -> 2.7n; footprint Socket_Strips:Socket_Strip_Straight_1x02_Pitch2.54mm -> Capacitors_SMD:C_0805_HandSoldering
- J1: footprint digikey-footprints:PinHeader_2x5_P2.54mm_Drill1.2mm -> rfid-footprints:jtag-header
- renumbered C16 to C10, C17 to C11, C18 to C12, C19 to C13, C20 to C14, C21 to C15, C32 to C16, C22 to C17, C3 to C2, C25 to C20, C26 to C21, C27 to C22, C28 to C23, C29 to C24, C30 to C25, C31 to C26, C4 to C3, C5 to C4, C8 to C5, C12 to C6, C13 to C7, C14 to C8, C15 to C9, D2 to D1, D4 to D2, D5 to D3, D6 to D4, D7 to D5, D8 to D6, FB2 to FB1, R3 to R1, R14 to R10, R25 to R11, R26 to R12, R15 to R13, R16 to R14, R17 to R15, R18 to R16, R19 to R17, R20 to R18, R21 to R19, R7 to R2, R22 to R20, R23 to R21, R24 to R22, R9 to R3, R10 to R4, R11 to R5, R12 to R6, R13 to R9, U3 to U2, U4 to U3, U6 to U5, U7 to U6
Connections:
- net +5V is gone; now on net +3V3: R11.2
- net DATA_IN_DIG is gone; now on net DATA_IN: U2.31 (PD6), U6.8
- net DATA_OUT is gone; now on net ANTENNA: U2.32 (PD7)
- net +3V3: now also U2.64 (AVCC), C18.1, R7.1, R8.1, U4.2 (OUT)
- net ANTENNA: now also C16.2, R13.1
- net CHARGE_MCP: now also BT1.1 (+), D5.2 (A), Q3.1 (B)
- net GND: now also C18.2, U4.1 (GND)
- net I2C_SCL: now also R7.2
- net I2C_SDA: now also R8.2
- net OC0: now also Q1.1 (B), Q2.1 (B)
- net USB_VBUS: now also Q3.2 (E)
- net VSUPPLY: now also U4.3 (IN)
- net at R13.2: now also Q1.2 (E), Q2.2 (E)
- net at R11.1: now also Q1.3 (C)
- net at R12.1: now also Q2.3 (C)
- net at D5.1 (K), S4.1: now also Q3.3 (C)
- net DATA_IN: now reaches U2.29 (PD4)
- net DATA_IN_AN: no longer names the net of C26.1, R21.1, R22.2, U6.10 (+), U6.7
- net DATA_IN_AN: no longer U2.61 (PF0)
- no-connect marks 14 -> 10
Other:
- note added: "Antenna (model as inductor)"
- note added: "Antenna Driver"
- note removed: "Antenna (model as 1mH inductor)"
- note removed: "Antenna Driver (Noelle)"
- note removed: "Antenna Load Switcher (Ian)"
- note removed: "LT8613 Charging Circuit (Ian)"
- note removed: "Use a socket for this cap\nrather than SMT footprint"
- moved on the sheet: C19
